Commit message: Added gazebo simulation for driving robot and other urdf modication

File: description/robot_core.xacro (robot description, xacro)
@@ -14,4 +14,7 @@
         <color rgba="0 0 0 1"/>
     </material>
+    <material name="yellow" >
+        <color rgba="1.0 1.0 0.0784313725490196 1.0" />
+    </material>
 <!-- BASE LINK -->
     <link name="base_link">
@@ -20,17 +23,17 @@
     <parent link="base_link"/>
     <child link="chassis"/>
-    <origin xyz="-0.25 0 0"/>
+    <origin xyz="0.25 0 0"/>
     </joint>
 <!-- CHASSIS -->
     <link name="chassis">
     <visual>
-        <origin xyz="0.35 0 0.075" rpy="0 0 0"/>
+        <origin xyz="-0.35 0 0.075" rpy="0 0 0"/>
         <geometry>
             <box size="0.7 0.38 0.15"/>
         </geometry>
-        <material name="white"/>
+        <material name="yellow"/>
     </visual>
     <collision>
-        <origin xyz="0.35 0 0.075" rpy="0 0 0"/>
+        <origin xyz="-0.35 0 0.075" rpy="0 0 0"/>
         <geometry>
             <box size="0.7 0.38 0.15"/>
@@ -38,7 +41,10 @@
     </collision>
     <xacro:inertial_box mass="0.5" x="0.7" y="0.38" z="0.15">
-        <origin xyz="0.35 0 0.075" rpy="0 0 0"/>
+        <origin xyz="-0.35 0 0.075" rpy="0 0 0"/>
     </xacro:inertial_box>
 </link>
+<gazebo reference="chassis">
+    <material>Gazebo/Yellow</material>
+</gazebo>
 <!-- LEFT WHEEL -->
 <joint name="left_wheel_joint" type="continuous">
@@ -64,4 +70,7 @@
     </xacro:inertial_cylinder>
 </link>
+<gazebo reference="left_wheel">
+    <material>Gazebo/Blue</material>
+</gazebo>
 <!-- RIGHT WHEEL -->
     <joint name="right_wheel_joint" type="continuous">
@@ -84,13 +93,16 @@
             <material name="blue"/>
         </collision>
-    </link>
     <xacro:inertial_cylinder mass="0.1" length="0.05" radius="0.0775">
         <origin xyz="0 0 0" rpy="0 0 0"/>
     </xacro:inertial_cylinder>
+</link>
+<gazebo reference="right_wheel">
+    <material>Gazebo/Blue</material>
+</gazebo>
 <!-- CASTER WHEEL -->
 <joint name="caster_wheel_joint" type="fixed">
     <parent link="chassis"/>
     <child link="caster_wheel"/>
-    <origin xyz="0.55 0 0" rpy="0 0 0"/>
+    <origin xyz="-0.55 0 0" rpy="0 0 0"/>
 </joint>
 <link name="caster_wheel">
@@ -111,3 +123,8 @@
     </xacro:inertial_sphere>
 </link>
+<gazebo reference="caster_wheel">
+    <material>Gazebo/Black</material>
+    <mu1 value="0.001"/>
+    <mu2 value="0.001"/>
+</gazebo>
 </robot>
